File: Circuit/NixieClock/NixieClock.kicad_sch (KiCad schematic)
At the start: 14 parts, among them J1 Conn_01x10, Q1 MMBTA42, U1 74141N, U2 74AHC595

Commit message: Set Conn Pin 4 as GND, Rule, and Board Shape
Connections:
- net GND: now also J1.7 (Pin_7)
Changed lines of the file:
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@@
+    (effects (font (size 1.27 1.27)) (justify left bottom))
+  )
+  (label "GND" (at 228.6 67.31 0)
     (effects (font (size 1.27 1.27)) (justify left bottom))
   )
